Commit message: transform added to wavefront

File: src/bot_sim/xacro/gazebo_my_laser.urdf.xacro (robot description, xacro)
@@ -35,8 +35,8 @@
     <xacro:property name="laser_length" value="0.05" />
     <xacro:property name="laser_radius" value="0.03" />
-    <xacro:property name="laser_x" value="0.0" />
-    <xacro:property name="laser_y" value="0.0" />
+    <xacro:property name="laser_x" value="0" />
+    <xacro:property name="laser_y" value="0" />
     <xacro:property name="laser_z" value="${support_length / 2 + laser_length / 2}" />
-    <xacro:property name="laser_m" value="0.1" />
+    <xacro:property name="laser_m" value="0.0" />
     <link name="laser">
         <visual>
